File: RFID_Shield.brd (EAGLE design)
At the start: 59.7 x 53.3 mm, 8 parts, among them J1 ARDUINO_R3_SHIELD, Q1 MMBT2222, U1 RFID

Commit message: Fixed missing VCC and GND connections.
Connections:
- net GND: now also J1.GND@0, J1.GND@1, J1.GND@2
- net VCC: now also J1.5V
Routing:
- net VCC: track 40.8 -> 69.5 mm
Changed lines of the file:
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@@
 <vertex x="0" y="29.21"/>
 </polygon>
+<contactref element="J1" pad="GND@2"/>
+<contactref element="J1" pad="GND@1"/>
+<contactref element="J1" pad="GND@0"/>
 </signal>
 <signal name="VCC">
@@
 <wire x1="50.8" y1="53.34" x2="50.8" y2="40.83" width="0.254" layer="1"/>
 <wire x1="50.8" y1="40.83" x2="50.99" y2="40.64" width="0.254" layer="1"/>
+<contactref element="J1" pad="5V"/>
+<wire x1="29.21" y1="29.21" x2="29.21" y2="33.02" width="0.254" layer="1"/>
+<wire x1="29.21" y1="33.02" x2="30.48" y2="34.29" width="0.254" layer="1"/>
+<wire x1="30.48" y1="34.29" x2="44.64" y2="34.29" width="0.254" layer="1"/>
+<wire x1="44.64" y1="34.29" x2="50.99" y2="40.64" width="0.254" layer="1"/>
 </signal>
 <signal name="LED">
